File: circut/solder_staion/solder_staion.kicad_pcb (KiCad board)
At the start: 2 copper layers, 23.6 x 25.5 mm, 24 parts, among them J1 Screw_Terminal_01x02, J3 Conn_01x01_Pin, J4 Conn_01x01_Pin, J5 Conn_01x01_Pin, J6 Conn_01x01_Pin, Q2 Si4162DY, U1 UC3842_SOIC8

Commit message: final v1
Parts:
- J3: footprint Connector_JST:JST_XH_B1B-XH-AM_1x01_P2.50mm_Vertical -> Connector_PinHeader_1.00mm:PinHeader_1x01_P1.00mm_Vertical
- J5, J6: footprint Connector_PinHeader_2.54mm:PinHeader_1x01_P2.54mm_Horizontal -> Connector_PinHeader_1.00mm:PinHeader_1x01_P1.00mm_Vertical
- moved J6 1.48 mm to (228.5, 88.2)
Routing:
- net T+: track 0.00 -> 7.75 mm
- net heater: track 23.5 -> 31.2 mm
- net T-: track 4.15 -> 10.1 mm
- net +24V: track 34.2 -> 38.5 mm
- net +5V: track 36.1 -> 35.3 mm
- added copper zone on B.Cu, net +24V
- added copper zone on B.Cu, net GND
- added copper zone on B.Cu, net heater
Other:
- board size 23.6 x 25.5 mm -> 23.6 x 25.9 mm
