File: circut/solder_staion/solder_staion.kicad_sch (KiCad schematic)
At the start: 21 parts, among them J1 Screw_Terminal_01x02, Q2 BUK9M17-30EX, U1 UC3842_SOIC8

Commit message: done_v1
Parts:
- removed Q2: BUK9M17-30EX, Package_TO_SOT_SMD:TDSON-8-1, symbol Transistor_FET:BUK9M17-30EX
- added J2: DIN-5, symbol Connector:DIN-5
- added J3: Conn_01x01_Pin, Connector_JST:JST_XH_B1B-XH-AM_1x01_P2.50mm_Vertical, symbol Connector:Conn_01x01_Pin
- added J4, J5, J6: Conn_01x01_Pin, Connector_PinHeader_2.54mm:PinHeader_1x01_P2.54mm_Horizontal, symbol Connector:Conn_01x01_Pin
- added Q2: Si4162DY, Package_SO:SOIC-8_3.9x4.9mm_P1.27mm, symbol Transistor_FET:Si4162DY
- C1, C2, C3, C4, C5, C6, C7, C8: footprint (none) -> Capacitor_SMD:C_1206_3216Metric_Pad1.33x1.80mm_HandSolder
- J1: footprint (none) -> TerminalBlock:TerminalBlock_MaiXu_MX126-5.0-02P_1x02_P5.00mm
- R1, R10, R11, R2, R3, R4, R6, R7: footprint (none) -> Resistor_SMD:R_1206_3216Metric_Pad1.30x1.75mm_HandSolder
- R5: now not fitted; now left out of the parts list
- RV1: footprint (none) -> Potentiometer_THT:Potentiometer_ACP_CA9-H3,8_Horizontal
Connections:
- net +24V: now also J2.2, J4.1 (Pin_1)
- net GND: now also Q2.1 (S), Q2.2 (S), Q2.3 (S)
- net T+: now also J2.4, J6.1 (Pin_1)
- net T-: now also J2.3, J3.1 (Pin_1)
- net at R4.2: now also Q2.4 (G)
- net heater: now reaches C7.2, R5.2
- net heater: now also J2.1, J5.1 (Pin_1), Q2.5 (D), Q2.6 (D), Q2.7 (D), Q2.8 (D)
Other:
- moved on the sheet: J1

Commit message: final v1
Connections:
- net T-: now also J2.5; no longer J2.3
Other:
- moved on the sheet: J1, J3
