File: lcd_ST/circut/lcd_soldring_staion/lcd_soldring_staion.kicad_sch (KiCad schematic)
At the start: 28 parts, among them J1 DIN-5, J1 Screw_Terminal_01x02, J2 Conn_01x05_Pin, J3 Conn_01x01_Pin, J4 Conn_01x01_Pin, J5 Conn_01x01_Pin, J6 Conn_01x01_Pin, J7 Conn_01x04_Pin, Q1 IRF7403, SW1 SW_Push, U1 PIC16F15223T-I/SL, U2 L7805, U3 LM358

Commit message: Update lcd_soldring_staion.kicad_sch
Connections:
- net GND: now also J7.2 (Pin_2); no longer J7.1 (Pin_1)
- net VCC: now also J7.1 (Pin_1); no longer J7.2 (Pin_2)
- net SCl renamed clk
- net SDA renamed dat
Changed lines of the file:
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@@
 		)
 	)
-	(global_label "SDA"
+	(global_label "dat"
 		(shape input)
 		(at 274.32 40.64 0)
@@
 		)
 		(property "Intersheetrefs" "${INTERSHEET_REFS}"
-			(at 280.8733 40.64 0)
+			(at 280.3289 40.64 0)
 			(effects
 				(font
@@
 		)
 	)
-	(global_label "SDA"
-		(shape input)
-		(at 232.41 83.82 0)
-		(fields_autoplaced yes)
-		(effects
-			(font
-				(size 1.27 1.27)
-			)
-			(justify left)
-		)
-		(property "Intersheetrefs" "${INTERSHEET_REFS}"
-			(at 238.9633 83.82 0)
-			(effects
-				(font
-					(size 1.27 1.27)
-				)
-				(justify left)
-				(hide yes)
-			)
-		)
-	)
 	(global_label "heater_gate"
 		(shape input)
@@
 		)
 	)
+	(global_label "clk"
+		(shape input)
+		(at 232.41 86.36 0)
+		(fields_autoplaced yes)
+		(effects
+			(font
+				(size 1.27 1.27)
+			)
+			(justify left)
+		)
+		(property "Intersheetrefs" "${INTERSHEET_REFS}"
+			(at 238.1771 86.36 0)
+			(effects
+				(font
+					(size 1.27 1.27)
+				)
+				(justify left)
+				(hide yes)
+			)
+		)
+	)
 	(global_label "T+"
 		(shape input)
@@
 		)
 	)
-	(global_label "SCl"
-		(shape input)
-		(at 232.41 86.36 0)
-		(fields_autoplaced yes)
-		(effects
-			(font
-				(size 1.27 1.27)
-			)
-			(justify left)
-		)
-		(property "Intersheetrefs" "${INTERSHEET_REFS}"
-			(at 238.5399 86.36 0)
-			(effects
-				(font
-					(size 1.27 1.27)
-				)
-				(justify left)
-				(hide yes)
-			)
-		)
-	)
 	(global_label "heater"
 		(shape input)
@@
 		)
 	)
-	(global_label "SCl"
+	(global_label "clk"
 		(shape input)
 		(at 274.32 43.18 0)
@@
 		)
 		(property "Intersheetrefs" "${INTERSHEET_REFS}"
-			(at 280.4499 43.18 0)
+			(at 280.0871 43.18 0)
 			(effects
 				(font
@@
 		)
 	)
+	(global_label "dat"
+		(shape input)
+		(at 232.41 83.82 0)
+		(fields_autoplaced yes)
+		(effects
+			(font
+				(size 1.27 1.27)
+			)
+			(justify left)
+		)
+		(property "Intersheetrefs" "${INTERSHEET_REFS}"
+			(at 238.4189 83.82 0)
+			(effects
+				(font
+					(size 1.27 1.27)
+				)
+				(justify left)
+				(hide yes)
+			)
+		)
+	)
 	(global_label "PGD"
 		(shape input)
@@
 	(symbol
 		(lib_id "power:GND")
-		(at 274.32 35.56 90)
+		(at 274.32 38.1 90)
 		(unit 1)
 		(exclude_from_sim no)
@@
 		(fields_autoplaced yes)
 		(property "Reference" "#PWR019"
-			(at 280.67 35.56 0)
+			(at 280.67 38.1 0)
 			(effects
 				(font
@@
 		)
 		(property "Value" "GND"
-			(at 278.13 35.5599 90)
+			(at 278.13 38.0999 90)
 			(effects
 				(font
@@
 		)
 		(property "Footprint" ""
-			(at 274.32 35.56 0)
+			(at 274.32 38.1 0)
 			(effects
 				(font
@@
 		)
 		(property "Datasheet" ""
-			(at 274.32 35.56 0)
+			(at 274.32 38.1 0)
 			(effects
 				(font
@@
 		)
 		(property "Description" "Power symbol creates a global label with name \"GND\" , ground"
-			(at 274.32 35.56 0)
+			(at 274.32 38.1 0)
 			(effects
 				(font
@@
 					(size 1.27 1.27)
 				)
+				(hide yes)
 			)
 		)
@@
 	(symbol
 		(lib_id "power:VCC")
-		(at 274.32 38.1 270)
+		(at 274.32 35.56 270)
 		(unit 1)
 		(exclude_from_sim no)
@@
 		(fields_autoplaced yes)
 		(property "Reference" "#PWR018"
-			(at 270.51 38.1 0)
+			(at 270.51 35.56 0)
 			(effects
 				(font
@@
 		)
 		(property "Value" "VCC"
-			(at 278.13 38.0999 90)
+			(at 278.13 35.5599 90)
 			(effects
 				(font
@@
 		)
 		(property "Footprint" ""
-			(at 274.32 38.1 0)
+			(at 274.32 35.56 0)
 			(effects
 				(font
@@
 		)
 		(property "Datasheet" ""
-			(at 274.32 38.1 0)
+			(at 274.32 35.56 0)
 			(effects
 				(font
@@
 		)
 		(property "Description" "Power symbol creates a global label with name \"VCC\""
-			(at 274.32 38.1 0)
+			(at 274.32 35.56 0)
 			(effects
 				(font

Commit message: k
Parts:
- removed Q1: IRF7403, Package_TO_SOT_SMD:Infineon_PG-HSOF-8-3_ThermalVias, symbol Transistor_FET:IRF7403
- added C10, C9: 100nf, Capacitor_SMD:C_1206_3216Metric_Pad1.33x1.80mm_HandSolder, symbol Device:C
- added Q2: Si4162DY, Package_SO:SOIC-8_3.9x4.9mm_P1.27mm, symbol Transistor_FET:Si4162DY
- added R10, R11: 120K, Resistor_SMD:R_1206_3216Metric_Pad1.30x1.75mm_HandSolder, symbol Device:R
- added R12, R8, R9: 1K, Resistor_SMD:R_1206_3216Metric_Pad1.30x1.75mm_HandSolder, symbol Device:R
- added R13: 1K, Resistor_SMD:R_1812_4532Metric_Pad1.30x3.40mm_HandSolder, symbol Device:R
- added unit 2 of U3
- C1: footprint (none) -> Capacitor_SMD:C_1206_3216Metric_Pad1.33x1.80mm_HandSolder
- J2: footprint (none) -> Connector_Molex:Molex_KK-254_AE-6410-05A_1x05_P2.54mm_Vertical
- J3: footprint Connector_JST:JST_XH_B1B-XH-AM_1x01_P2.50mm_Vertical -> Connector_PinHeader_2.54mm:PinHeader_1x01_P2.54mm_Vertical
- J4, J5, J6: footprint Connector_PinHeader_2.54mm:PinHeader_1x01_P2.54mm_Horizontal -> Connector_PinHeader_2.54mm:PinHeader_1x01_P2.54mm_Vertical
- J7: footprint (none) -> Connector:FanPinHeader_1x04_P2.54mm_Vertical
- R1, R2, R3, R4, R5, R6, R7: footprint (none) -> Resistor_SMD:R_1206_3216Metric_Pad1.30x1.75mm_HandSolder
- RV1: footprint (none) -> Potentiometer_THT:Potentiometer_ACP_CA9-H2,5_Horizontal
- SW1: footprint (none) -> Button_Switch_SMD:SW_DIP_SPSTx01_Slide_6.7x4.1mm_W6.73mm_P2.54mm_LowProfile_JPin
- U1: footprint SOIC14_SL_MCH -> pic16f15223:SOIC14_SL_MCH
- U2: footprint (none) -> Package_TO_SOT_SMD:TO-252-3_TabPin2
- U3: footprint (none) -> Package_SO:SOIC-8_5.3x6.2mm_P1.27mm
- renumbered J1 to J44
Connections:
- net 24v is gone; now on net +24V: R1.1
- net GND: now also RV1.3, C10.2, C9.2, R10.1, R13.1, R9.1; no longer RV1.1
- net VCC: now also RV1.1; no longer RV1.3
- net heater: now also Q2.5 (D), Q2.6 (D), Q2.7 (D), Q2.8 (D)
- net at R7.2: now also Q2.4 (G)
- net current: now reaches U1.7 (RC3)
- net current: now also C10.1, R12.2
- new net: R11.1, R8.2, U3.5 (+)
- new net: R10.2, R9.2, U3.6 (-)
- new net: R11.2, R12.1, U3.7
- new net c+: C9.1, Q2.1 (S), Q2.2 (S), Q2.3 (S), R13.2, R8.1
Other:
- moved on the sheet: C4, C5, R2, R3, R4, R5, R6, U3A

Commit message: done v0
Connections:
- net GND: now also C9.1, R8.1; no longer C9.2, R9.1
- net T+: now also C4.2, R4.1; no longer C4.1, R2.1
- net T-: now also C4.1, R2.1; no longer C4.2, R4.1
- net c+: now also C9.2, R9.1; no longer C9.1, R8.1
- net at R11.1, R8.2: now also U3.6 (-); no longer U3.5 (+)
- net at R10.2, R9.2: now also U3.5 (+); no longer U3.6 (-)
- net at R4.2, R5.2: now also U3.3 (+); no longer U3.2 (-)
- net at R2.2, R3.1: now also U3.2 (-); no longer U3.3 (+)
Other:
- moved on the sheet: R2, R4, R5

Commit message: V2_PCB EDITING
Parts:
- added D1: LED, LED_SMD:LED_0805_2012Metric_Pad1.15x1.40mm_HandSolder, symbol Device:LED
- added J8: Conn_01x04_Pin, Connector:FanPinHeader_1x04_P2.54mm_Vertical, symbol Connector:Conn_01x04_Pin
- added R14, R15, R16: 1K, Resistor_SMD:R_1206_3216Metric_Pad1.30x1.75mm_HandSolder, symbol Device:R
- added SW2: RotaryEncoder_Switch, symbol Device:RotaryEncoder_Switch
Connections:
- net GND: now also D1.1 (K), J8.3 (Pin_3), SW2.C, SW2.S2
- net VCC: now also J8.4 (Pin_4), R14.1, R15.1
- net TX: now reaches U1.11 (RA2)
- net TX: now also J8.2 (Pin_2)
- net at U1.6 (RC4): now also R16.2
- net RX: now reaches U1.8 (RC2)
- net RX: now also J8.1 (Pin_1)
- net PGC renamed B
- net B: now also R14.2, SW2.B
- net PGD renamed A
- net A: now also R15.2, SW2.A
- net temp_set renamed ClC
- net ClC: now also SW2.S1
- new net: D1.2 (A), R16.1

Commit message: pcb v2
Parts:
- removed SW2: RotaryEncoder_Switch, symbol Device:RotaryEncoder_Switch
- added J9: Conn_01x04_Pin, Connector:FanPinHeader_1x04_P2.54mm_Vertical, symbol Connector:Conn_01x04_Pin
- D1: footprint LED_SMD:LED_0805_2012Metric_Pad1.15x1.40mm_HandSolder -> LED_SMD:LED_1210_3225Metric_Pad1.42x2.65mm_HandSolder
- R1, R10, R11, R12, R14, R15, R16, R2, R3, R4, R5, R6, R8, R9: footprint Resistor_SMD:R_1206_3216Metric_Pad1.30x1.75mm_HandSolder -> Resistor_SMD:R_0805_2012Metric_Pad1.20x1.40mm_HandSolder
- R13: footprint Resistor_SMD:R_1812_4532Metric_Pad1.30x3.40mm_HandSolder -> Resistor_SMD:R_0805_2012Metric_Pad1.20x1.40mm_HandSolder
- R7: value 1K -> 0.02
Connections:
- net A: now also J9.2 (Pin_2)
- net B: now also J9.1 (Pin_1)
- net ClC: now also J9.4 (Pin_4)
- net GND: now also J9.3 (Pin_3)
Other:
- moved on the sheet: R14, R15

Commit message: pcb v2
Parts:
- added J10: Conn_01x03_Pin, symbol Connector:Conn_01x03_Pin
- J9, R15: now not fitted; now left out of the parts list
- R1: value 330 -> 50; footprint Resistor_SMD:R_0805_2012Metric_Pad1.20x1.40mm_HandSolder -> Resistor_THT:R_Axial_DIN0207_L6.3mm_D2.5mm_P7.62mm_Horizontal
- R14, RV1: now not fitted
Connections:
- net ClC: now also J10.2 (Pin_2)
- net GND: now also J10.3 (Pin_3); no longer D1.1 (K)
- net VCC: now also J10.1 (Pin_1)
- net at R16.2: no longer U1.6 (RC4)
Other:
- moved on the sheet: C2, D1, R16

Commit message: pcbing
Parts:
- J4: now not fitted; now left out of the parts list
- J7, J8: footprint Connector:FanPinHeader_1x04_P2.54mm_Vertical -> Connector:01x04_fat_pins
- R14: now left out of the parts list
- U3: footprint Package_SO:SOIC-8_5.3x6.2mm_P1.27mm -> Package_SO:SOIC-8_3.9x4.9mm_P1.27mm
Connections:
- net TX: now also U1.9 (RC1); no longer U1.11 (RA2)
- net clk: now also U1.10 (RC0); no longer U1.9 (RC1)
- net dat: now also U1.11 (RA2); no longer U1.10 (RC0)
Changed lines of the file:
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@@
 		)
 	)
-	(global_label "TX"
-		(shape input)
-		(at 232.41 81.28 0)
-		(fields_autoplaced yes)
-		(effects
-			(font
-				(size 1.27 1.27)
-			)
-			(justify left)
-		)
-		(property "Intersheetrefs" "${INTERSHEET_REFS}"
-			(at 237.5723 81.28 0)
-			(effects
-				(font
-					(size 1.27 1.27)
-				)
-				(justify left)
-				(hide yes)
-			)
-		)
-	)
 	(global_label "heater"
 		(shape input)
@@
 		)
 	)
-	(global_label "clk"
+	(global_label "A"
 		(shape input)
-		(at 232.41 86.36 0)
+		(at 240.03 76.2 0)
 		(fields_autoplaced yes)
 		(effects
@@
 		)
 		(property "Intersheetrefs" "${INTERSHEET_REFS}"
-			(at 238.1771 86.36 0)
+			(at 244.1038 76.2 0)
 			(effects
 				(font
@@
 		)
 	)
-	(global_label "A"
+	(global_label "temp_set"
 		(shape input)
-		(at 240.03 76.2 0)
+		(at 156.21 78.74 180)
+		(fields_autoplaced yes)
+		(effects
+			(font
+				(size 1.27 1.27)
+			)
+			(justify right)
+		)
+		(property "Intersheetrefs" "${INTERSHEET_REFS}"
+			(at 144.7582 78.74 0)
+			(effects
+				(font
+					(size 1.27 1.27)
+				)
+				(justify right)
+				(hide yes)
+			)
+		)
+	)
+	(global_label "TEMP"
+		(shape input)
+		(at 132.08 120.65 0)
 		(fields_autoplaced yes)
 		(effects
@@
 		)
 		(property "Intersheetrefs" "${INTERSHEET_REFS}"
-			(at 244.1038 76.2 0)
+			(at 139.9032 120.65 0)
 			(effects
 				(font
@@
 		)
 	)
-	(global_label "temp_set"
+	(global_label "c+"
 		(shape input)
-		(at 156.21 78.74 180)
+		(at 187.96 127 180)
 		(fields_autoplaced yes)
 		(effects
@@
 		)
 		(property "Intersheetrefs" "${INTERSHEET_REFS}"
-			(at 144.7582 78.74 0)
+			(at 182.3138 127 0)
 			(effects
 				(font
@@
 		)
 	)
-	(global_label "TEMP"
+	(global_label "TX"
 		(shape input)
-		(at 132.08 120.65 0)
+		(at 232.41 86.36 0)
 		(fields_autoplaced yes)
 		(effects
@@
 		)
 		(property "Intersheetrefs" "${INTERSHEET_REFS}"
-			(at 139.9032 120.65 0)
+			(at 237.5723 86.36 0)
 			(effects
 				(font
@@
 		)
 	)
-	(global_label "c+"
+	(global_label "TEMP"
 		(shape input)
-		(at 187.96 127 180)
+		(at 156.21 76.2 180)
 		(fields_autoplaced yes)
 		(effects
@@
 		)
 		(property "Intersheetrefs" "${INTERSHEET_REFS}"
-			(at 182.3138 127 0)
+			(at 148.3868 76.2 0)
 			(effects
 				(font
@@
 		)
 	)
-	(global_label "TEMP"
+	(global_label "dat"
 		(shape input)
-		(at 156.21 76.2 180)
+		(at 232.41 81.28 0)
 		(fields_autoplaced yes)
 		(effects
@@
 				(size 1.27 1.27)
 			)
-			(justify right)
+			(justify left)
 		)
 		(property "Intersheetrefs" "${INTERSHEET_REFS}"
-			(at 148.3868 76.2 0)
+			(at 238.4189 81.28 0)
 			(effects
 				(font
 					(size 1.27 1.27)
 				)
-				(justify right)
+				(justify left)
+				(hide yes)
+			)
+		)
+	)
+	(global_label "clk"
+		(shape input)
+		(at 232.41 83.82 0)
+		(fields_autoplaced yes)
+		(effects
+			(font
+				(size 1.27 1.27)
+			)
+			(justify left)
+		)
+		(property "Intersheetrefs" "${INTERSHEET_REFS}"
+			(at 238.1771 83.82 0)
+			(effects
+				(font
+					(size 1.27 1.27)
+				)
+				(justify left)
 				(hide yes)
 			)
@@
 		)
 	)
-	(global_label "dat"
-		(shape input)
-		(at 232.41 83.82 0)
-		(fields_autoplaced yes)
-		(effects
-			(font
-				(size 1.27 1.27)
-			)
-			(justify left)
-		)
-		(property "Intersheetrefs" "${INTERSHEET_REFS}"
-			(at 238.4189 83.82 0)
-			(effects
-				(font
-					(size 1.27 1.27)
-				)
-				(justify left)
-				(hide yes)
-			)
-		)
-	)
 	(global_label "PGD"
 		(shape input)
@@
 			)
 		)
-		(property "Footprint" "Package_SO:SOIC-8_5.3x6.2mm_P1.27mm"
+		(property "Footprint" "Package_SO:SOIC-8_3.9x4.9mm_P1.27mm"
 			(at 119.38 153.67 0)
 			(effects
@@
 			)
 		)
-		(property "Footprint" "Connector:FanPinHeader_1x04_P2.54mm_Vertical"
+		(property "Footprint" "Connector:01x04_fat_pins"
 			(at 270.51 20.32 0)
 			(effects
@@
 		(at 243.84 60.96 90)
 		(unit 1)
-		(exclude_from_sim no)
-		(in_bom yes)
-		(on_board yes)
+		(exclude_from_sim yes)
+		(in_bom no)
+		(on_board no)
 		(dnp yes)
 		(property "Reference" "R14"
@@
 			)
 		)
-		(property "Footprint" "Connector:FanPinHeader_1x04_P2.54mm_Vertical"
+		(property "Footprint" "Connector:01x04_fat_pins"
 			(at 269.24 38.1 0)
 			(effects
@@
 			)
 		)
-		(property "Footprint" "Package_SO:SOIC-8_5.3x6.2mm_P1.27mm"
+		(property "Footprint" "Package_SO:SOIC-8_3.9x4.9mm_P1.27mm"
 			(at 26.67 85.09 0)
 			(effects
@@
 			)
 		)
-		(property "Footprint" "Package_SO:SOIC-8_5.3x6.2mm_P1.27mm"
+		(property "Footprint" "Package_SO:SOIC-8_3.9x4.9mm_P1.27mm"
 			(at 116.84 120.65 0)
 			(effects
@@
 		(unit 1)
 		(exclude_from_sim no)
-		(in_bom yes)
-		(on_board yes)
-		(dnp no)
+		(in_bom no)
+		(on_board no)
+		(dnp yes)
 		(property "Reference" "J4"
 			(at 254 126.365 0)

Commit message: da
Parts:
- J10: footprint (none) -> Connector:FanPinHeader_1x03_P2.54mm_Vertical
Connections:
- net ClC: now also J10.1 (Pin_1); no longer J10.2 (Pin_2)
- net VCC: now also J10.2 (Pin_2); no longer J10.1 (Pin_1)
Other:
- moved on the sheet: C6
Changed lines of the file:
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@@
 	)
 	(junction
+		(at 254 88.9)
+		(diameter 0)
+		(color 0 0 0 0)
+	)
+	(junction
 		(at 92.71 124.46)
 		(diameter 0)
@@
 	(wire
 		(pts
+			(xy 254 96.52) (xy 255.27 96.52)
+		)
+		(stroke
+			(width 0)
+			(type default)
+		)
+	)
+	(wire
+		(pts
 			(xy 41.91 64.77) (xy 43.18 64.77)
 		)
@@
 	(wire
 		(pts
+			(xy 265.43 100.33) (xy 259.08 100.33)
+		)
+		(stroke
+			(width 0)
+			(type default)
+		)
+	)
+	(wire
+		(pts
 			(xy 270.51 88.9) (xy 269.24 88.9)
 		)
@@
 	(wire
 		(pts
-			(xy 270.51 91.44) (xy 262.89 91.44)
+			(xy 270.51 93.98) (xy 262.89 93.98)
 		)
 		(stroke
@@
 	(wire
 		(pts
+			(xy 270.51 91.44) (xy 265.43 91.44)
+		)
+		(stroke
+			(width 0)
+			(type default)
+		)
+	)
+	(wire
+		(pts
 			(xy 139.7 81.28) (xy 156.21 81.28)
 		)
@@
 	(wire
 		(pts
-			(xy 259.08 92.71) (xy 259.08 93.98)
+			(xy 259.08 92.71) (xy 259.08 100.33)
+		)
+		(stroke
+			(width 0)
+			(type default)
+		)
+	)
+	(wire
+		(pts
+			(xy 262.89 88.9) (xy 262.89 93.98)
 		)
 		(stroke
@@
 	(wire
 		(pts
-			(xy 247.65 60.96) (xy 264.16 60.96)
+			(xy 265.43 91.44) (xy 265.43 100.33)
 		)
 		(stroke
@@
 	(wire
 		(pts
-			(xy 270.51 93.98) (xy 259.08 93.98)
+			(xy 247.65 60.96) (xy 264.16 60.96)
 		)
 		(stroke
@@
 	(wire
 		(pts
+			(xy 254 88.9) (xy 255.27 88.9)
+		)
+		(stroke
+			(width 0)
+			(type default)
+		)
+	)
+	(wire
+		(pts
 			(xy 240.03 55.88) (xy 240.03 58.42)
 		)
@@
 	(wire
 		(pts
-			(xy 252.73 88.9) (xy 255.27 88.9)
+			(xy 252.73 88.9) (xy 254 88.9)
 		)
 		(stroke
@@
 	(wire
 		(pts
-			(xy 262.89 91.44) (xy 262.89 88.9)
-		)
-		(stroke
-			(width 0)
-			(type default)
-		)
-	)
-	(wire
-		(pts
 			(xy 92.71 124.46) (xy 97.79 124.46)
 		)
@@
 			)
 		)
-		(property "Footprint" ""
+		(property "Footprint" "Connector:FanPinHeader_1x03_P2.54mm_Vertical"
 			(at 275.59 91.44 0)
 			(effects
@@
 	(symbol
 		(lib_id "Device:C")
-		(at 255.27 92.71 0)
+		(at 254 92.71 0)
 		(unit 1)
 		(exclude_from_sim no)
@@
 		(dnp no)
 		(property "Reference" "C6"
-			(at 259.08 91.4399 0)
+			(at 257.81 91.4399 0)
 			(effects
 				(font
@@
 		)
 		(property "Value" "100nf"
-			(at 247.65 93.98 0)
+			(at 246.38 93.98 0)
 			(effects
 				(font
@@
 		)
 		(property "Footprint" "Capacitor_SMD:C_1206_3216Metric_Pad1.33x1.80mm_HandSolder"
-			(at 256.2352 96.52 0)
+			(at 254.9652 96.52 0)
 			(effects
 				(font
@@
 		)
 		(property "Datasheet" "~"
-			(at 255.27 92.71 0)
+			(at 254 92.71 0)
 			(effects
 				(font
@@
 		)
 		(property "Description" "Unpolarized capacitor"
-			(at 255.27 92.71 0)
+			(at 254 92.71 0)
 			(effects
 				(font
