File: lcd_ST/circut/lcd_soldring_staion/lcd_soldring_staion.kicad_pcb (KiCad board)
At the start: 2 copper layers, 45 x 42.6 mm, 35 parts, among them J10 Conn_01x03_Pin, J2 Conn_01x05_Pin, J3 Conn_01x01_Pin, J44 Screw_Terminal_01x02, J5 Conn_01x01_Pin, J6 Conn_01x01_Pin, J7 Conn_01x04_Pin, J8 Conn_01x04_Pin, Q2 Si4162DY, SW1 SW_Push, U1 PIC16F15223T-I/SL, U2 L7805, U3 LM358

Commit message: final_final
Routing:
- net TEMP: track 27.7 -> 28.6 mm
Other:
- board size 45 x 42.6 mm -> 45 x 44.4 mm
